File: rxnWheel/rxnWheel.kicad_sch (KiCad schematic)
At the start: 13 parts

Commit message: kiran changes
Parts:
- removed C1: C, symbol Device:C
- removed C2: (no value), symbol Device:C
- removed R1, R3: R_Small, symbol Device:R_Small
- removed R2: (no value), symbol Device:R_Small
- removed TH1: (no value), symbol Device:Thermistor_NTC
- added C? (x3): (no value), symbol Device:C
- added R? (x4): (no value), symbol Device:R
- D1: value (none) -> DIODE
- IC1: value (none) -> TB9061AFNG,EL; footprint (none) -> SOP65P760X160-24N
- L1: value (none) -> L
Connections:
- net GND: now also C?.1, C?.2, C?.2, R?.1, R?.2
- net at IC1.3 (IPC): now also C?.2
- net ASIG: now reaches IC1.5 (SFCF)
- net ASIG: now also IC1.22 (ASIG), R?.1, R?.2
- net at IC1.1 (PSIG): now also C?.1, R?.2, R?.2
- net VReg: now reaches IC1.23 (VREG), IC1.24 (VDD)
- net VReg: now also C?.1, R?.1
- new net PWM_IN: R?.1

Commit message: .
Parts:
- removed C4: C, symbol Device:C
- removed L1: L, symbol Device:L
- added C1, C10, C8, C9: 1uF, Capacitor_SMD:C_0805_2012Metric, symbol Device:C
- added C17, C18: 20pF, Capacitor_SMD:C_0805_2012Metric, symbol Device:C
- added C6: 0.01uF, Capacitor_SMD:C_0805_2012Metric, symbol Device:C
- added C7: 0.1uF, Capacitor_SMD:C_0805_2012Metric, symbol Device:C
- added Q1: IRF7458, Package_SO:SOIC-8_3.9x4.9mm_P1.27mm, symbol Transistor_FET:IRF7404
- added R10: 4K, Resistor_SMD:R_0805_2012Metric, symbol Device:R
- added R13, R3, R6, R7: 10K, Resistor_SMD:R_0805_2012Metric, symbol Device:R
- added R15: 1K, Resistor_SMD:R_0805_2012Metric, symbol Device:R
- added R8: 3m, Resistor_SMD:R_1206_3216Metric, symbol Device:R
- added R9: 6K, Resistor_SMD:R_0805_2012Metric, symbol Device:R
- added U1: ATmega328-P, Package_DIP:DIP-28_W7.62mm, symbol MCU_Microchip_ATmega:ATmega328-P
- added U2: MAX4373F, Package_SO:SO-8_3.9x4.9mm_P1.27mm, symbol symbols:MAX4373F
- added Y1: 16MHz, Crystal:Crystal_HC49-4H_Vertical, symbol Device:Crystal
- C2: renamed from C?; value (none) -> 1nF; footprint (none) -> Capacitor_SMD:C_0805_2012Metric
- C3: value C -> 1uF; footprint (none) -> Capacitor_SMD:C_0805_2012Metric
- C4: renamed from C?; value (none) -> 0.47 uF; footprint (none) -> Capacitor_SMD:C_0805_2012Metric
- C5: renamed from C?; value (none) -> 0.1uF; footprint (none) -> Capacitor_SMD:C_0805_2012Metric
- IC1: value TB9061AFNG,EL -> TB9061AFNG; footprint SOP65P760X160-24N -> TB9061AFNG:SOP65P760X160-24N
- R1: renamed from R?; value (none) -> 100; footprint (none) -> Resistor_SMD:R_0805_2012Metric
- R11, R12, R2: renamed from R?; value (none) -> 10K; footprint (none) -> Resistor_SMD:R_0805_2012Metric
- R4, R5: value R_Small -> 10K; footprint (none) -> Resistor_SMD:R_0805_2012Metric
Connections:
- net +BATT: now also Q1.1 (S), Q1.2 (S), Q1.3 (S), R3.1
- net GND: now also IC1.6 (SLA), IC1.7 (CW_CCW), C1.2, C10.2, C17.1, C18.1, C6.1, C7.1, C8.2, C9.2, R10.2, U1.22 (GND), U1.8 (GND), U2.4 (GND)
- net WAVE_CMP: now also C7.2
- net U_N: now reaches IC1.10 (OUTUN)
- net V_N: now reaches IC1.11 (OUTVN)
- net W_N: now reaches IC1.12 (OUTWN)
- net U_P: now reaches IC1.13 (OUTUP)
- net V_P: now reaches IC1.14 (OUTVP)
- net W_P: now reaches IC1.15 (OUTWP)
- net U_W: now reaches IC1.17 (WAVE_U)
- net V_W: now reaches IC1.18 (WAVE_V)
- net W_W: now reaches IC1.19 (WAVE_W)
- net at IC1.21 (OCDET): now also C6.2, R15.1
- net SHUTOFF: now reaches IC1.4 (DIS)
- net OUTFG: now reaches IC1.8 (OUTFG)
- net Batt-Reg renamed I_SENSE
- net I_SENSE: now also R15.2
- new net: Q1.4 (G), R3.2, R6.2, U2.6 (COUT1)
- new net: Q1.5 (D), Q1.6 (D), Q1.7 (D), Q1.8 (D), R8.2, U2.8 (RS+)
- new net: R6.1, R7.1, U2.1 (Vcc)
- new net: R7.2, U2.5 (~{RESET})
- new net: C18.2, Y1.2
- new net: R10.1, R9.2, U2.3 (CIN1)
- new net: C17.2, U1.9 (XTAL1/PB6), Y1.1
- new net +5V: C1.1, R13.2, U1.20 (AVCC), U1.7 (VCC)
- new net BTL1: U1.17 (PB3)
- new net BTL2: U1.18 (PB4)
- new net BTL3: U1.19 (PB5)
- new net I_MOTOR_TELEM: R9.1, U2.2 (OUT)
- new net RESET: R13.1, U1.1 (~{RESET}/PC6)
- new net VBUS: C10.1, C8.1, C9.1, R8.1, U2.7 (RS-)
Other:
- added sheet U (NP_switch\NP_switch.kicad_sch)
- added sheet V (NP_switch\NP_switch.kicad_sch)
- added sheet W (NP_switch\NP_switch.kicad_sch)
- moved on the sheet: C5, R4, R5

Commit message: Commit
CoMmMMmMMMmits
Parts:
- removed Q1: IRF7458, Package_SO:SOIC-8_3.9x4.9mm_P1.27mm, symbol Transistor_FET:IRF7404
- removed R10: 4K, Resistor_SMD:R_0805_2012Metric, symbol Device:R
- removed R3, R6, R7: 10K, Resistor_SMD:R_0805_2012Metric, symbol Device:R
- removed R8: 3m, Resistor_SMD:R_1206_3216Metric, symbol Device:R
- removed R9: 6K, Resistor_SMD:R_0805_2012Metric, symbol Device:R
- removed U2: MAX4373F, Package_SO:SO-8_3.9x4.9mm_P1.27mm, symbol symbols:MAX4373F
- added C?: 0.1uF, Capacitor_SMD:C_0805_2012Metric, symbol Device:C
- added Q? (x2): 2N7002, Package_TO_SOT_SMD:SOT-23, symbol Transistor_FET:2N7002
- added Q?: IRF7458, Package_SO:SOIC-8_3.9x4.9mm_P1.27mm, symbol Transistor_FET:IRF7404
- added R? (x4): 10K, Resistor_SMD:R_0805_2012Metric, symbol Device:R
- added R?: 3m, Resistor_SMD:R_1206_3216Metric, symbol Device:R
- added R?: 3K, Resistor_SMD:R_0805_2012Metric, symbol Device:R
- added R?: 9.5K, Resistor_SMD:R_0805_2012Metric, symbol Device:R
- added U?: MAX4373F, Package_SO:SO-8_3.9x4.9mm_P1.27mm, symbol symbols:MAX4373F
Connections:
- net SHUTOFF is gone; now on net GND: IC1.4 (DIS)
- net +BATT: now also C?.1, Q?.1 (S), Q?.2 (S), Q?.3 (S), R?.1, R?.1, R?.1, U?.1 (Vcc)
- net GND: now also U1.14 (PB0), C?.2, Q?.2 (S), R?.1, R?.2, R?.2, U?.4 (GND)
- net I_MOTOR_TELEM: now also U1.23 (PC0), R?.1, U?.2 (OUT)
- net PWM_IN: now also U1.11 (PD5)
- net VBUS: now also R?.1, U?.7 (RS-)
- net RSTMTRVOCP: now reaches U1.12 (PD6)
- net RSTMTRVOCP: now also R?.2, U?.5 (~{RESET})
- net RSTMTRV: now reaches U1.13 (PD7)
- net RSTMTRV: now also Q?.1 (G)
- net DRN_MTR: now reaches U1.15 (PB1)
- new net: Q?.2 (S), Q?.3 (D)
- new net: R?.1, R?.2, U?.3 (CIN1)
- new net: Q?.1 (G), R?.2, U?.6 (COUT1)
- new net: Q?.5 (D), Q?.6 (D), Q?.7 (D), Q?.8 (D), R?.2, U?.8 (RS+)
- new net: Q?.3 (D), Q?.4 (G), R?.2

Commit message: HANDS
fix fix hands hands
Parts:
- added R?: 100, Resistor_SMD:R_0805_2012Metric, symbol Device:R
Connections:
- net DRN_MTR: now also R?.1; no longer U1.15 (PB1)
- net GND: no longer IC1.4 (DIS), R?.2, U1.14 (PB0)
- new net: R?.2, U1.15 (PB1)
- new net SHUTOFF: IC1.4 (DIS), R?.2, U1.14 (PB0)
Other:
- moved on the sheet: C1

Commit message: minor changes
Other:
- sheet U: file NP_switch\NP_switch.kicad_sch -> NP_switch/NP_switch.kicad_sch
- sheet V: file NP_switch\NP_switch.kicad_sch -> NP_switch/NP_switch.kicad_sch
- sheet W: file NP_switch\NP_switch.kicad_sch -> NP_switch/NP_switch.kicad_sch
Changed lines of the file:
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@@
   )
   (symbol (lib_id "Device:R") (at 67.31 64.77 90) (unit 1)
-    (in_bom yes) (on_board yes) (fields_autoplaced)
-    (property "Reference" "R13" (id 0) (at 67.31 58.42 90))
-    (property "Value" "10K" (id 1) (at 67.31 60.96 90))
+    (in_bom yes) (on_board yes)
+    (property "Reference" "R13" (id 0) (at 67.31 62.23 90))
+    (property "Value" "10K" (id 1) (at 67.31 64.77 90))
     (property "Footprint" "Resistor_SMD:R_0805_2012Metric" (id 2) (at 67.31 66.548 90)
       (effects (font (size 1.27 1.27)) hide)
@@
       (effects (font (size 1.27 1.27)) (justify left bottom))
     )
-    (property "Sheet file" "NP_switch\\NP_switch.kicad_sch" (id 1) (at 224.79 93.2946 0)
+    (property "Sheet file" "NP_switch/NP_switch.kicad_sch" (id 1) (at 224.79 93.2946 0)
       (effects (font (size 1.27 1.27)) (justify left top))
     )
@@
       (effects (font (size 1.27 1.27)) (justify left bottom))
     )
-    (property "Sheet file" "NP_switch\\NP_switch.kicad_sch" (id 1) (at 224.79 150.4446 0)
+    (property "Sheet file" "NP_switch/NP_switch.kicad_sch" (id 1) (at 224.79 150.4446 0)
       (effects (font (size 1.27 1.27)) (justify left top))
     )
@@
       (effects (font (size 1.27 1.27)) (justify left bottom))
     )
-    (property "Sheet file" "NP_switch\\NP_switch.kicad_sch" (id 1) (at 224.79 123.7746 0)
+    (property "Sheet file" "NP_switch/NP_switch.kicad_sch" (id 1) (at 224.79 123.7746 0)
       (effects (font (size 1.27 1.27)) (justify left top))
     )
@@
       (reference "#PWR?") (unit 1) (value "+BATT") (footprint "")
     )
+    (path "/ac4486ff-84d5-4133-ba84-b6c4de1ddb19/4669e73e-b1c6-4295-bc4c-92f45e5fd735"
+      (reference "#PWR?") (unit 1) (value "GND") (footprint "")
+    )
     (path "/8e485e19-4b91-45a4-88b2-6a19a5a0013f/4669e73e-b1c6-4295-bc4c-92f45e5fd735"
       (reference "#PWR?") (unit 1) (value "GND") (footprint "")
@@
       (reference "#PWR?") (unit 1) (value "GND") (footprint "")
     )
-    (path "/ac4486ff-84d5-4133-ba84-b6c4de1ddb19/4669e73e-b1c6-4295-bc4c-92f45e5fd735"
-      (reference "#PWR?") (unit 1) (value "GND") (footprint "")
-    )
     (path "/5acf29ab-dac4-4eb0-ac95-016cd6b4d9ae"
       (reference "#PWR?") (unit 1) (value "GND") (footprint "")
@@
       (reference "Q?") (unit 1) (value "IRF7458") (footprint "Package_SO:SOIC-8_3.9x4.9mm_P1.27mm")
     )
+    (path "/ac4486ff-84d5-4133-ba84-b6c4de1ddb19/c5ec54f0-0d08-4954-a314-8acf9272ac84"
+      (reference "Q?") (unit 1) (value "Si4162DY") (footprint "Package_SO:SOIC-8_3.9x4.9mm_P1.27mm")
+    )
+    (path "/a7e11de0-b987-453e-9e08-30a2e3d4892c/c5ec54f0-0d08-4954-a314-8acf9272ac84"
+      (reference "Q?") (unit 1) (value "Si4162DY") (footprint "Package_SO:SOIC-8_3.9x4.9mm_P1.27mm")
+    )
     (path "/8e485e19-4b91-45a4-88b2-6a19a5a0013f/c5ec54f0-0d08-4954-a314-8acf9272ac84"
       (reference "Q?") (unit 1) (value "Si4162DY") (footprint "Package_SO:SOIC-8_3.9x4.9mm_P1.27mm")
     )
-    (path "/ac4486ff-84d5-4133-ba84-b6c4de1ddb19/c5ec54f0-0d08-4954-a314-8acf9272ac84"
-      (reference "Q?") (unit 1) (value "Si4162DY") (footprint "Package_SO:SOIC-8_3.9x4.9mm_P1.27mm")
-    )
-    (path "/a7e11de0-b987-453e-9e08-30a2e3d4892c/c5ec54f0-0d08-4954-a314-8acf9272ac84"
-      (reference "Q?") (unit 1) (value "Si4162DY") (footprint "Package_SO:SOIC-8_3.9x4.9mm_P1.27mm")
-    )

Commit message: Brake
commmit
Parts:
- added C? (x3): 1uF, Capacitor_SMD:C_0805_2012Metric, symbol Device:C
- added D?: BPW20RF, symbol Device:D_Photo
- added Q?: 2N3904, Package_TO_SOT_THT:TO-92_Inline, symbol Transistor_BJT:2N3904
- added R? (x2): 1K, Resistor_SMD:R_0805_2012Metric, symbol Device:R
- added R?: 3m, Resistor_SMD:R_0805_2012Metric, symbol Device:R
Connections:
- net +5V: now also D?.1 (K), Q?.3 (C)
- net GND: now also R?.1, R?.1, R?.1
- net I_SENSE: now also R?.2
- net VReg: now also IC1.22 (ASIG)
- net MTR_FRQ: now reaches U1.16 (PB2)
- net MTR_FRQ: now also Q?.1 (E), R?.2
- net ASIG: no longer names the net of R11.2, R12.1
- net ASIG: no longer IC1.22 (ASIG), IC1.5 (SFCF)
- new net: D?.2 (A), Q?.2 (B), R?.2
- new net SFCF: IC1.5 (SFCF)
- new net U/BRK_OUT: C?.1, C?.1
- new net V/BRK_OUT: C?.2, C?.2
- new net W/BRK_OUT: C?.1, C?.2
Other:
- sheet U ports: added BRK_OUT; removed none
- sheet V ports: added BRK_OUT; removed none
- sheet W ports: added BRK_OUT; removed none
- moved on the sheet: R12

Commit message: LED
led
Parts:
- added D9: LED, TB9061AFNG:2x_jumper, symbol Device:LED
- added R34: 1K, Resistor_SMD:R_0805_2012Metric, symbol Device:R
- D8: renamed from D?; footprint (none) -> TB9061AFNG:2x_jumper
- R11: value 10K -> 3K
- R12: value 10K -> 7K
- gave numbers to parts that had none: 20
Connections:
- net +5V: now also D9.2 (A)
- net GND: now also R34.1
- net SFCF: now also R11.2, R12.1
- new net: D9.1 (K), R34.2
Other:
- moved on the sheet: R11

Commit message: cleanup and corrections
Parts:
- removed C19, C5, C7: 0.1uF, Capacitor_SMD:C_0805_2012Metric, symbol Device:C
- removed C6: 0.01uF, Capacitor_SMD:C_0805_2012Metric, symbol Device:C
- removed D1: DIODE, symbol Simulation_SPICE:DIODE
- removed IC1: TB9061AFNG, TB9061AFNG:SOP65P760X160-24N, symbol TB9061AFNG:TB9061AFNG,EL
- removed Q1, Q9: 2N7002, Package_TO_SOT_SMD:SOT-23, symbol Transistor_FET:2N7002
- removed Q8: IRF7458, Package_SO:SOIC-8_3.9x4.9mm_P1.27mm, symbol Transistor_FET:IRF7404
- removed R1: 100, Resistor_SMD:R_0805_2012Metric, symbol Device:R
- removed R11: 3K, Resistor_SMD:R_0805_2012Metric, symbol Device:R
- removed R12: 7K, Resistor_SMD:R_0805_2012Metric, symbol Device:R
- removed R15: 1K, Resistor_SMD:R_0805_2012Metric, symbol Device:R
- removed R2: 10K, Resistor_SMD:R_0805_2012Metric, symbol Device:R
- removed R35: 3m, Resistor_SMD:R_0805_2012Metric, symbol Device:R
- removed R4, R5: 10K, Resistor_SMD:R_0805_2012Metric, symbol Device:R_Small
- removed U2: MAX4373F, Package_SO:SO-8_3.9x4.9mm_P1.27mm, symbol symbols:MAX4373F
- added R40: 10K, Resistor_SMD:R_0805_2012Metric, symbol Device:R
- added R41, R42, R43: 33K, Resistor_SMD:R_0805_2012Metric, symbol Device:R
- added TP? (x3): (no value), symbol Connector:TestPoint
- added U2: ATmega328-P, Package_DIP:DIP-28_W7.62mm, symbol MCU_Microchip_ATmega:ATmega328-P
- added Y2: 16MHz, Crystal:Crystal_HC49-4H_Vertical, symbol Device:Crystal
- C2: value 1nF -> 20pF
- C3: value 1uF -> 20pF
- C4: value 0.47 uF -> 1uF
- R10: value 9.5K -> 10K
- R14: value 3K -> 10K
- R6, R8: value 10K -> 33K
- R9: value 3m -> 33K; footprint Resistor_SMD:R_1206_3216Metric -> Resistor_SMD:R_0805_2012Metric
Connections:
- net +5V: now also C4.1, R3.2, U2.20 (AVCC), U2.7 (VCC)
- net GND: now also C2.1, C3.1, C4.2, R10.1, R14.1, R40.1, U2.22 (GND), U2.8 (GND); no longer C2.2, C3.2, C4.1, R14.2
- net U_MTR: now also R41.1, TP?.1
- net U_N: now also U2.19 (PB5)
- net U_P: now also U2.16 (PB2)
- net VBUS: no longer R9.1
- net V_MTR: now also R42.1, TP?.1
- net V_N: now also U2.17 (PB3)
- net V_P: now also U2.14 (PB0)
- net W_MTR: now also R43.1, TP?.1
- net W_N: now also U2.18 (PB4)
- net W_P: now also U2.15 (PB1)
- net A2: now reaches R10.2
- net A2: now also R6.1, R41.2, U2.25 (PC2); no longer R14.1
- net at R6.2: now also R8.2, R9.2, U2.12 (PD6)
- net at C18.2, Y1.2: now also U1.10 (XTAL2/PB7)
- net PWM_CONTROL: now reaches U1.2 (PD0)
- net PWM_CONTROL: now also U2.2 (PD0)
- removed net +BATT: R3.1, R6.1, R8.1
- net DRN_MTR renamed DRV_MTR
- net I_MOTOR_TELEM: no longer names the net of U1.23 (PC0)
- net I_MOTOR_TELEM: no longer R10.1
- net PWM_IN: no longer names the net of U1.11 (PD5)
- net RSTMTRV: no longer names the net of U1.13 (PD7)
- net RSTMTRVOCP: no longer names the net of U1.12 (PD6)
- net RSTMTRVOCP: no longer R8.2
- new net: R3.1, U2.1 (~{RESET}/PC6)
- new net: C3.2, U2.10 (XTAL2/PB7), Y2.2
- new net: C2.2, U2.9 (XTAL1/PB6), Y2.1
- new net A0: R40.2, R43.2, R9.1, U2.23 (PC0)
- new net A1: R14.2, R42.2, R8.1, U2.24 (PC1)
Other:
- sheet U ports: added none; removed I_SENSE
- sheet V ports: added none; removed I_SENSE
- sheet W ports: added none; removed I_SENSE
- moved on the sheet: C10, C20, C21, C22, C8, C9
