File: rxnWheel/NP_switch/NP_switch.kicad_sch (KiCad schematic)
At the start: 16 parts, among them Q3 Si4162DY

Commit message: corrected capacitors
Parts:
- removed C?: 0.1uF, Capacitor_SMD:C_0805_2012Metric, symbol Device:C
- removed C? (x4): 22uF, Capacitor_SMD:C_1210_3225Metric, symbol Device:C
- C?: value 22uF -> (none)
